File: fmu_v1.kicad_sch (KiCad schematic)
At the start: 0 parts

Commit message: da
Other:
- company: (none) -> TampanTech
- title: (none) -> Architecture
Changed lines of the file:
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@@
 	(generator_version "8.0")
 	(paper "A4")
+	(title_block
+		(title "Architecture")
+		(date "2024-09-08")
+		(rev "1")
+		(company "TampanTech")
+		(comment 1 "Drone Flight Management Unit")
+	)
 	(sheet
 		(at 55.88 151.13)
