File: memory.kicad_sch (KiCad schematic)
At the start: 18 parts, among them J14 USB_B_Micro, J18 Micro_SD_Card_Det1, Q7 Si2301CDS-T1-GE3

Commit message: da
Other:
- company: (none) -> TampanTech
- title: (none) -> Memory
Changed lines of the file:
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@@
 	(generator_version "8.0")
 	(paper "A4")
+	(title_block
+		(title "Memory")
+		(date "2024-09-08")
+		(rev "1")
+		(company "TampanTech")
+		(comment 1 "Drone Flight Management Unit")
+	)
 	(junction
 		(at 127 95.25)
