File: USB.kicad_sch (KiCad schematic)
At the start: 57 parts, among them J1 Conn_01x07, J4 Conn_01x04, J5 Conn_01x05, Q1 Q_NPN_BEC, Q2 Q_NPN_BEC, Q3 Q_NPN_BEC, SW1 EVQ-P7A01P, Y2 16.00 Mhz

Commit message: da
Other:
- company: (none) -> TampanTech
- title: (none) -> USBConn
Changed lines of the file:
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@@
 	(generator_version "8.0")
 	(paper "A4")
+	(title_block
+		(title "USBConn")
+		(date "2024-09-08")
+		(rev "1")
+		(company "TampanTech")
+		(comment 1 "Drone Flight Management Unit")
+	)
 	(junction
 		(at 203.2 127)

Commit message: change label to global
Connections:
- net  I2C0_SDA_EXTERNAL renamed _I2C0_SDA_EXTERNAL
- net  LED_AMBER renamed _LED_AMBER

Commit message: change label to global
Parts:
- C47, C50: footprint 3PAD_NFM15PC_0402_MUR -> (none)
- SW1: footprint EVQ_P7_PAN -> (none)
Changed lines of the file:
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@@
 			)
 		)
-		(property "Footprint" "3PAD_NFM15PC_0402_MUR"
+		(property "Footprint" ""
 			(at 177.8 27.94 0)
 			(effects
@@
 			)
 		)
-		(property "Footprint" "EVQ_P7_PAN"
+		(property "Footprint" ""
 			(at 93.98 180.34 0)
 			(effects
@@
 			)
 		)
-		(property "Footprint" "3PAD_NFM15PC_0402_MUR"
+		(property "Footprint" ""
 			(at 218.44 102.87 0)
 			(effects
