File: conn2.kicad_sch (KiCad schematic)
At the start: 31 parts, among them J11 Conn_01x06, J12 HDR_3x9, U5 NTB0104GU12_115, U6 NTB0104GU12_115, U7 NTB0104GU12_115, U8 BMI088, U9 BMM150

Commit message: da
Other:
- company: (none) -> TampanTech
- title: (none) -> Connector2
Changed lines of the file:
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@@
 	(generator_version "8.0")
 	(paper "A4")
+	(title_block
+		(title "Connector2")
+		(date "2024-09-08")
+		(rev "1")
+		(company "TampanTech")
+		(comment 1 "Drone Flight Management Unit")
+	)
 	(junction
 		(at 154.94 165.1)

Commit message: change label to global
Parts:
- C63: footprint 3PAD_NFM15PC_0402_MUR -> (none)
- U5, U7: footprint XQFN12_SOT1174-1_NEX_NXP -> (none)
Changed lines of the file:
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@@
 			)
 		)
-		(property "Footprint" "XQFN12_SOT1174-1_NEX_NXP"
+		(property "Footprint" ""
 			(at 60.96 49.53 0)
 			(effects
@@
 			)
 		)
-		(property "Footprint" "3PAD_NFM15PC_0402_MUR"
+		(property "Footprint" ""
 			(at 149.86 35.56 0)
 			(effects
@@
 			)
 		)
-		(property "Footprint" "XQFN12_SOT1174-1_NEX_NXP"
+		(property "Footprint" ""
 			(at 31.75 171.45 0)
 			(effects
