File: ethernet.kicad_sch (KiCad schematic)
At the start: 66 parts, among them J15 Conn_01x02, J16 BM04B-GHS-TBT(LF)(SN)(N), Q6 Si2301CDS-T1-GE3, U15 TJA1100HNZ, U16 TJA1042TK-3, Y3 25MHz

Commit message: da
Other:
- company: (none) -> TampanTech
- title: (none) -> Ethernet
Changed lines of the file:
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@@
 	(generator_version "8.0")
 	(paper "A4")
+	(title_block
+		(title "Ethernet")
+		(rev "1")
+		(company "TampanTech")
+		(comment 1 "Drone Flight Management Unit")
+	)
 	(junction
 		(at 231.14 57.15)

Commit message: change label to global
Connections:
- net  RMII_MDIO renamed _RMII_MDIO

Commit message: change label to global
Parts:
- CR1: footprint SOT143B_NEX -> (none)
Changed lines of the file:
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@@
 			)
 		)
-		(property "Footprint" "SOT143B_NEX"
+		(property "Footprint" ""
 			(at 217.17 77.47 0)
 			(effects
