File: sensoric.kicad_sch (KiCad schematic)
At the start: 27 parts, among them J13 SM02B-GHS-TB, U10 ICM-42688-P, U11 BMP280, U12 W25X40CLUXIG_TR, U13 SE050C1HQ1/Z01SCZ, U14 FM25V02A-GTR

Commit message: da
Other:
- company: (none) -> TampanTech
- title: (none) -> Sensoric
Changed lines of the file:
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@@
 	(generator_version "8.0")
 	(paper "A4")
+	(title_block
+		(title "Sensoric")
+		(date "2024-09-08")
+		(rev "1")
+		(company "TampanTech")
+		(comment 1 "Drone Flight Management Unit")
+	)
 	(junction
 		(at 135.89 55.88)

Commit message: change label to global
Parts:
- J13: footprint CONN_SM02B-GHS_JST -> (none)
- U13: footprint HX2QFN20_SOT1969_3X3_NXP -> (none)
Changed lines of the file:
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@@
 			)
 		)
-		(property "Footprint" "CONN_SM02B-GHS_JST"
+		(property "Footprint" ""
 			(at 109.22 83.82 0)
 			(effects
@@
 			)
 		)
-		(property "Footprint" "HX2QFN20_SOT1969_3X3_NXP"
+		(property "Footprint" ""
 			(at 140.97 99.06 0)
 			(effects
